Commit message: name set to solo12; prev was GazeboSystem

File: solo12_description/urdf/solo12.ros2control.xacro (robot description, xacro)
@@ -3,5 +3,6 @@
   <xacro:macro name="solo12_ros2control" params="prefix" >
     <!-- ROS2_CONTROL tag name: -->
-    <xacro:property name="name" value="GazeboSystem"/>
+    <xacro:property name="name" value="solo12"/>
+    <!--<xacro:property name="name" value="GazeboSystem"/>-->
     <!-- ===== Gazebo ROS2_CONTROL plugin ===== -->
     <!--
@@ -26,12 +27,9 @@
                 <param name="max">${pi}</param>
             </command_interface>
-            <command_interface name="velocity">
-                <param name="min">-3.15</param>
-                <param name="max">3.15</param>
-            </command_interface>
             <state_interface name="position">
                 <param name="initial_value">0.0</param>
             </state_interface>
             <state_interface name="velocity"/>
+            <state_interface name="effort"/>
         </joint>
         <!-- FL_HFE -->
@@ -41,12 +39,9 @@
                 <param name="max">${pi}</param>
             </command_interface>
-            <command_interface name="velocity">
-                <param name="min">-3.15</param>
-                <param name="max">3.15</param>
-            </command_interface>
             <state_interface name="position">
                 <param name="initial_value">0.0</param>
             </state_interface>
             <state_interface name="velocity"/>
+            <state_interface name="effort"/>
         </joint>
         <!-- FL_KFE -->
@@ -56,12 +51,9 @@
                 <param name="max">${pi}</param>
             </command_interface>
-            <command_interface name="velocity">
-                <param name="min">-3.15</param>
-                <param name="max">3.15</param>
-            </command_interface>
             <state_interface name="position">
                 <param name="initial_value">0.0</param>
             </state_interface>
             <state_interface name="velocity"/>
+            <state_interface name="effort"/>
         </joint>
         <!-- FR_HAA -->
@@ -71,12 +63,9 @@
                 <param name="max">${pi}</param>
             </command_interface>
-            <command_interface name="velocity">
-                <param name="min">-3.15</param>
-                <param name="max">3.15</param>
-            </command_interface>
             <state_interface name="position">
                 <param name="initial_value">0.0</param>
             </state_interface>
             <state_interface name="velocity"/>
+            <state_interface name="effort"/>
         </joint>
         <!-- FR_HFE -->
@@ -86,12 +75,9 @@
                 <param name="max">${pi}</param>
             </command_interface>
-            <command_interface name="velocity">
-                <param name="min">-3.15</param>
-                <param name="max">3.15</param>
-            </command_interface>
             <state_interface name="position">
                 <param name="initial_value">0.0</param>
             </state_interface>
             <state_interface name="velocity"/>
+            <state_interface name="effort"/>
         </joint>
         <!-- FR_KFE -->
@@ -101,12 +87,9 @@
                 <param name="max">${pi}</param>
             </command_interface>
-            <command_interface name="velocity">
-                <param name="min">-3.15</param>
-                <param name="max">3.15</param>
-            </command_interface>
             <state_interface name="position">
                 <param name="initial_value">0.0</param>
             </state_interface>
             <state_interface name="velocity"/>
+            <state_interface name="effort"/>
         </joint>
         <!-- HL_HAA -->
@@ -116,12 +99,9 @@
                 <param name="max">${pi}</param>
             </command_interface>
-            <command_interface name="velocity">
-                <param name="min">-3.15</param>
-                <param name="max">3.15</param>
-            </command_interface>
             <state_interface name="position">
                 <param name="initial_value">0.0</param>
             </state_interface>
             <state_interface name="velocity"/>
+            <state_interface name="effort"/>
         </joint>
         <!-- HL_HFE -->
@@ -131,12 +111,9 @@
                 <param name="max">${pi}</param>
             </command_interface>
-            <command_interface name="velocity">
-                <param name="min">-3.15</param>
-                <param name="max">3.15</param>
-            </command_interface>
             <state_interface name="position">
                 <param name="initial_value">0.0</param>
             </state_interface>
             <state_interface name="velocity"/>
+            <state_interface name="effort"/>
         </joint>
         <!-- HL_KFE -->
@@ -146,12 +123,9 @@
                 <param name="max">${pi}</param>
             </command_interface>
-            <command_interface name="velocity">
-                <param name="min">-3.15</param>
-                <param name="max">3.15</param>
-            </command_interface>
             <state_interface name="position">
                 <param name="initial_value">0.0</param>
             </state_interface>
             <state_interface name="velocity"/>
+            <state_interface name="effort"/>
         </joint>
         <!-- HR_HAA -->
@@ -161,12 +135,9 @@
                 <param name="max">${pi}</param>
             </command_interface>
-            <command_interface name="velocity">
-                <param name="min">-3.15</param>
-                <param name="max">3.15</param>
-            </command_interface>
             <state_interface name="position">
                 <param name="initial_value">0.0</param>
             </state_interface>
             <state_interface name="velocity"/>
+            <state_interface name="effort"/>
         </joint>
         <!-- HR_HFE -->
@@ -176,12 +147,9 @@
                 <param name="max">${pi}</param>
             </command_interface>
-            <command_interface name="velocity">
-                <param name="min">-3.15</param>
-                <param name="max">3.15</param>
-            </command_interface>
             <state_interface name="position">
                 <param name="initial_value">0.0</param>
             </state_interface>
             <state_interface name="velocity"/>
+            <state_interface name="effort"/>
         </joint>
         <!-- HR_KFE -->
@@ -191,12 +159,9 @@
                 <param name="max">${pi}</param>
             </command_interface>
-            <command_interface name="velocity">
-                <param name="min">-3.15</param>
-                <param name="max">3.15</param>
-            </command_interface>
             <state_interface name="position">
                 <param name="initial_value">0.0</param>
             </state_interface>
             <state_interface name="velocity"/>
+            <state_interface name="effort"/>
         </joint>
     </ros2_control>
