Commit message: added dummy_link; use_gazebo_classic arg

File: solo12_description/urdf/solo12_robot.urdf.xacro (robot description, xacro)
@@ -1,20 +1,21 @@
 <?xml version="1.0"?>
 <robot xmlns:xacro="http://www.ros.org/wiki/xacro" name="solo12">
-    <!--
-    <xacro:arg  name="ros2_controllers_file_path"
-                default="$(find solo12_gazebo)/config/controllers.yaml"/>
-    -->
-    <xacro:include  filename="$(find solo12_description)/urdf/solo12.gazebo.xacro" />
-    <xacro:solo12_gazebo
-            prefix="" />
-    <!-- common gazebo stuff -->
-    <!--<xacro:include  filename="$(find solo12_description)/urdf/common.gazebo.xacro" />-->
-    <!-- solo -->
-    <xacro:include  filename="$(find solo12_description)/urdf/solo12.urdf.xacro" />
-    <xacro:solo12_quadruped
-            prefix="" />
-    <!-- ROS2_CONTROL -->
-    <xacro:include  filename="$(find solo12_description)/urdf/solo12.ros2control.xacro" />
-    <xacro:solo12_ros2control
-            prefix="" />
+        <xacro:arg name="prefix" default="" />
+        <xacro:arg name="use_gazebo_classic" default="false" />
+        <!-- Import solo12 macro -->
+        <xacro:include  filename="$(find solo12_description)/urdf/solo12.urdf.xacro" />
+        <!-- Import solo12 ros2_control description -->
+        <xacro:include  filename="$(find solo12_description)/urdf/solo12.ros2_control.xacro" />
+        <!-- common gazebo stuff -->
+        <!--<xacro:include  filename="$(find solo12_description)/urdf/common.gazebo.xacro" />-->
+        <link name="dummy_link" />
+        <xacro:solo12_quadruped
+          parent="dummy_link" prefix="$(arg prefix)" />
+        <xacro:solo12_ros2_control
+          name="solo12" prefix="$(arg prefix)" use_gazebo_classic="$(arg use_gazebo_classic)" />
+        <xacro:if value="$(arg use_gazebo_classic)">
+          <!-- Import Gazebo Classic definitions + plugin -->
+          <xacro:include filename="$(find solo12_description)/urdf/solo12.gazebo.xacro" />
+          <xacro:solo12_gazebo prefix="$(arg prefix)" />
+        </xacro:if>
 </robot>
