Commit message: added gazebo ros2_control plugin

File: solo12_description/urdf/solo12.gazebo.xacro (robot description, xacro)
@@ -3,5 +3,4 @@
     <xacro:macro name="solo12_gazebo" params="prefix">
         <!-- ===== Gazebo ROS2_CONTROL plugin ===== -->
-        <!--
         <gazebo>
             <plugin filename="libgazebo_ros2_control.so" name="gazebo_ros2_control">
@@ -9,174 +8,173 @@
             </plugin>
         </gazebo>
-        -->
-        <gazebo reference="world" />
         <gazebo reference="${prefix}base_link">
+            <!-- <turnGravityOff>false</turnGravityOff>
             <selfCollide>true</selfCollide>
-            <mu1 value="0.0"/>
-            <mu2 value="0.0"/>
             <kp value="10000000.0"/>
             <kd value="1.0"/>
-            <material>Gazebo/Grey</material>
-            <turnGravityOff>false</turnGravityOff>
+            <fdir1 value="1 0 0"/> -->
+            <mu1 value="0.2"/>
+            <mu2 value="0.2"/>
+            <material>Gazebo/DarkGrey</material>
         </gazebo>
         <gazebo reference="${prefix}FL_SHOULDER">
+            <!-- <turnGravityOff>false</turnGravityOff>
             <selfCollide>true</selfCollide>
-            <mu1 value="1.0"/>
-            <mu2 value="1.0"/>
             <kp value="10000000.0"/>
             <kd value="1.0"/>
-            <!-- <fdir1 value="1 0 0"/> -->
+            <fdir1 value="1 0 0"/> -->
+            <mu1 value="0.2"/>
+            <mu2 value="0.2"/>
             <material>Gazebo/Grey</material>
-            <turnGravityOff>false</turnGravityOff>
         </gazebo>
         <gazebo reference="${prefix}FL_UPPER_LEG">
+            <!-- <turnGravityOff>false</turnGravityOff>
             <selfCollide>true</selfCollide>
-            <mu1 value="1.0"/>
-            <mu2 value="1.0"/>
             <kp value="10000000.0"/>
             <kd value="1.0"/>
-            <!-- <fdir1 value="1 0 0"/> -->
+            <fdir1 value="1 0 0"/> -->
+            <mu1 value="0.2"/>
+            <mu2 value="0.2"/>
             <material>Gazebo/Grey</material>
-            <turnGravityOff>false</turnGravityOff>
         </gazebo>
         <gazebo reference="${prefix}FL_LOWER_LEG">
+            <!-- <turnGravityOff>false</turnGravityOff>
             <selfCollide>true</selfCollide>
-            <mu1 value="1.0"/>
-            <mu2 value="1.0"/>
             <kp value="10000000.0"/>
             <kd value="1.0"/>
-            <!-- <fdir1 value="1 0 0"/> -->
+            <fdir1 value="1 0 0"/> -->
+            <mu1 value="0.2"/>
+            <mu2 value="0.2"/>
             <material>Gazebo/Grey</material>
-            <turnGravityOff>false</turnGravityOff>
         </gazebo>
         <gazebo reference="${prefix}FL_FOOT">
+            <!-- <turnGravityOff>false</turnGravityOff>
             <selfCollide>true</selfCollide>
-            <mu1 value="1.0"/>
-            <mu2 value="1.0"/>
             <kp value="10000000.0"/>
             <kd value="1.0"/>
-            <!-- <fdir1 value="1 0 0"/> -->
+            <fdir1 value="1 0 0"/> -->
+            <mu1 value="0.2"/>
+            <mu2 value="0.2"/>
             <material>Gazebo/Grey</material>
-            <turnGravityOff>false</turnGravityOff>
         </gazebo>
         <gazebo reference="${prefix}FR_SHOULDER">
+            <!-- <turnGravityOff>false</turnGravityOff>
             <selfCollide>true</selfCollide>
-            <mu1 value="1.0"/>
-            <mu2 value="1.0"/>
             <kp value="10000000.0"/>
             <kd value="1.0"/>
-            <!-- <fdir1 value="1 0 0"/> -->
+            <fdir1 value="1 0 0"/> -->
+            <mu1 value="0.2"/>
+            <mu2 value="0.2"/>
             <material>Gazebo/Grey</material>
-            <turnGravityOff>false</turnGravityOff>
         </gazebo>
         <gazebo reference="${prefix}FR_UPPER_LEG">
+            <!-- <turnGravityOff>false</turnGravityOff>
             <selfCollide>true</selfCollide>
-            <mu1 value="1.0"/>
-            <mu2 value="1.0"/>
             <kp value="10000000.0"/>
             <kd value="1.0"/>
-            <!-- <fdir1 value="1 0 0"/> -->
+            <fdir1 value="1 0 0"/> -->
+            <mu1 value="0.2"/>
+            <mu2 value="0.2"/>
             <material>Gazebo/Grey</material>
-            <turnGravityOff>false</turnGravityOff>
         </gazebo>
         <gazebo reference="${prefix}FR_LOWER_LEG">
+            <!-- <turnGravityOff>false</turnGravityOff>
             <selfCollide>true</selfCollide>
-            <mu1 value="1.0"/>
-            <mu2 value="1.0"/>
             <kp value="10000000.0"/>
             <kd value="1.0"/>
-            <!-- <fdir1 value="1 0 0"/> -->
+            <fdir1 value="1 0 0"/> -->
+            <mu1 value="0.2"/>
+            <mu2 value="0.2"/>
             <material>Gazebo/Grey</material>
-            <turnGravityOff>false</turnGravityOff>
         </gazebo>
         <gazebo reference="${prefix}FR_FOOT">
+            <!-- <turnGravityOff>false</turnGravityOff>
             <selfCollide>true</selfCollide>
-            <mu1 value="1.0"/>
-            <mu2 value="1.0"/>
             <kp value="10000000.0"/>
             <kd value="1.0"/>
-            <!-- <fdir1 value="1 0 0"/> -->
+            <fdir1 value="1 0 0"/> -->
+            <mu1 value="0.2"/>
+            <mu2 value="0.2"/>
             <material>Gazebo/Grey</material>
-            <turnGravityOff>false</turnGravityOff>
         </gazebo>
         <gazebo reference="${prefix}HL_SHOULDER">
+            <!-- <turnGravityOff>false</turnGravityOff>
             <selfCollide>true</selfCollide>
-            <mu1 value="1.0"/>
-            <mu2 value="1.0"/>
             <kp value="10000000.0"/>
             <kd value="1.0"/>
-            <!-- <fdir1 value="1 0 0"/> -->
+            <fdir1 value="1 0 0"/> -->
+            <mu1 value="0.2"/>
+            <mu2 value="0.2"/>
             <material>Gazebo/Grey</material>
-            <turnGravityOff>false</turnGravityOff>
         </gazebo>
         <gazebo reference="${prefix}HL_UPPER_LEG">
+            <!-- <turnGravityOff>false</turnGravityOff>
             <selfCollide>true</selfCollide>
-            <mu1 value="1.0"/>
-            <mu2 value="1.0"/>
             <kp value="10000000.0"/>
             <kd value="1.0"/>
-            <!-- <fdir1 value="1 0 0"/> -->
+            <fdir1 value="1 0 0"/> -->
+            <mu1 value="0.2"/>
+            <mu2 value="0.2"/>
             <material>Gazebo/Grey</material>
-            <turnGravityOff>false</turnGravityOff>
         </gazebo>
         <gazebo reference="${prefix}HL_LOWER_LEG">
+            <!-- <turnGravityOff>false</turnGravityOff>
             <selfCollide>true</selfCollide>
-            <mu1 value="1.0"/>
-            <mu2 value="1.0"/>
             <kp value="10000000.0"/>
             <kd value="1.0"/>
-            <!-- <fdir1 value="1 0 0"/> -->
+            <fdir1 value="1 0 0"/> -->
+            <mu1 value="0.2"/>
+            <mu2 value="0.2"/>
             <material>Gazebo/Grey</material>
-            <turnGravityOff>false</turnGravityOff>
         </gazebo>
         <gazebo reference="${prefix}HL_FOOT">
+            <!-- <turnGravityOff>false</turnGravityOff>
             <selfCollide>true</selfCollide>
-            <mu1 value="1.0"/>
-            <mu2 value="1.0"/>
             <kp value="10000000.0"/>
             <kd value="1.0"/>
-            <!-- <fdir1 value="1 0 0"/> -->
+            <fdir1 value="1 0 0"/> -->
+            <mu1 value="0.2"/>
+            <mu2 value="0.2"/>
             <material>Gazebo/Grey</material>
-            <turnGravityOff>false</turnGravityOff>
         </gazebo>
         <gazebo reference="${prefix}HR_SHOULDER">
+            <!-- <turnGravityOff>false</turnGravityOff>
             <selfCollide>true</selfCollide>
-            <mu1 value="1.0"/>
-            <mu2 value="1.0"/>
             <kp value="10000000.0"/>
             <kd value="1.0"/>
-            <!-- <fdir1 value="1 0 0"/> -->
+            <fdir1 value="1 0 0"/> -->
+            <mu1 value="0.2"/>
+            <mu2 value="0.2"/>
             <material>Gazebo/Grey</material>
-            <turnGravityOff>false</turnGravityOff>
         </gazebo>
         <gazebo reference="${prefix}HR_UPPER_LEG">
+            <!-- <turnGravityOff>false</turnGravityOff>
             <selfCollide>true</selfCollide>
-            <mu1 value="1.0"/>
-            <mu2 value="1.0"/>
             <kp value="10000000.0"/>
             <kd value="1.0"/>
-            <!-- <fdir1 value="1 0 0"/> -->
+            <fdir1 value="1 0 0"/> -->
+            <mu1 value="0.2"/>
+            <mu2 value="0.2"/>
             <material>Gazebo/Grey</material>
-            <turnGravityOff>false</turnGravityOff>
         </gazebo>
         <gazebo reference="${prefix}HR_LOWER_LEG">
+            <!-- <turnGravityOff>false</turnGravityOff>
             <selfCollide>true</selfCollide>
-            <mu1 value="1.0"/>
-            <mu2 value="1.0"/>
             <kp value="10000000.0"/>
             <kd value="1.0"/>
-            <!-- <fdir1 value="1 0 0"/> -->
+            <fdir1 value="1 0 0"/> -->
+            <mu1 value="0.2"/>
+            <mu2 value="0.2"/>
             <material>Gazebo/Grey</material>
-            <turnGravityOff>false</turnGravityOff>
         </gazebo>
         <gazebo reference="${prefix}HR_FOOT">
+            <!-- <turnGravityOff>false</turnGravityOff>
             <selfCollide>true</selfCollide>
-            <mu1 value="1.0"/>
-            <mu2 value="1.0"/>
             <kp value="10000000.0"/>
             <kd value="1.0"/>
-            <!-- <fdir1 value="1 0 0"/> -->
+            <fdir1 value="1 0 0"/> -->
+            <mu1 value="0.2"/>
+            <mu2 value="0.2"/>
             <material>Gazebo/Grey</material>
-            <turnGravityOff>false</turnGravityOff>
         </gazebo>
     </xacro:macro>

Commit message: modified gazebo link properties

File: solo12_description/urdf/solo12.gazebo.xacro (robot description, xacro)
@@ -9,172 +9,194 @@
         </gazebo>
         <gazebo reference="${prefix}base_link">
-            <!-- <turnGravityOff>false</turnGravityOff>
-            <selfCollide>true</selfCollide>
-            <kp value="10000000.0"/>
-            <kd value="1.0"/>
-            <fdir1 value="1 0 0"/> -->
-            <mu1 value="0.2"/>
-            <mu2 value="0.2"/>
-            <material>Gazebo/DarkGrey</material>
+            <mu1>0.05</mu1>
+            <mu2>0.05</mu2>
+            <!-- <kp>1000000.0</kp>
+            <kd>1.0</kd> -->
+            <maxVel>0.01</maxVel>
+            <material>Gazebo/DarkGrey </material>
         </gazebo>
         <gazebo reference="${prefix}FL_SHOULDER">
-            <!-- <turnGravityOff>false</turnGravityOff>
-            <selfCollide>true</selfCollide>
-            <kp value="10000000.0"/>
-            <kd value="1.0"/>
-            <fdir1 value="1 0 0"/> -->
-            <mu1 value="0.2"/>
-            <mu2 value="0.2"/>
-            <material>Gazebo/Grey</material>
+            <mu1>0.2</mu1>
+            <mu2>0.2</mu2>
+            <kp value="2147483647.0"/>
+            <kd value="1.0"/>
+            <maxVel>0.01</maxVel>
+            <self_collide>1</self_collide>
+            <material>Gazebo/PioneerBody</material>
         </gazebo>
         <gazebo reference="${prefix}FL_UPPER_LEG">
-            <!-- <turnGravityOff>false</turnGravityOff>
-            <selfCollide>true</selfCollide>
-            <kp value="10000000.0"/>
-            <kd value="1.0"/>
-            <fdir1 value="1 0 0"/> -->
-            <mu1 value="0.2"/>
-            <mu2 value="0.2"/>
-            <material>Gazebo/Grey</material>
+            <mu1>0.2</mu1>
+            <mu2>0.2</mu2>
+            <kp value="2147483647.0"/>
+            <kd value="1.0"/>
+            <maxVel>0.01</maxVel>
+            <self_collide>1</self_collide>
+            <material>Gazebo/Orange</material>
+            <!-- <implicitSpringDamper>1</implicitSpringDamper>
+            <springStiffness>100</springStiffness> -->
         </gazebo>
         <gazebo reference="${prefix}FL_LOWER_LEG">
-            <!-- <turnGravityOff>false</turnGravityOff>
-            <selfCollide>true</selfCollide>
-            <kp value="10000000.0"/>
-            <kd value="1.0"/>
-            <fdir1 value="1 0 0"/> -->
-            <mu1 value="0.2"/>
-            <mu2 value="0.2"/>
-            <material>Gazebo/Grey</material>
+            <mu1>0.2</mu1>
+            <mu2>0.2</mu2>
+            <fdir1>1 0 0</fdir1>
+            <kp>2147483647.0</kp>
+            <kd>1.0</kd>
+            <maxVel>0.01</maxVel>
+            <self_collide>1</self_collide>
+            <material>Gazebo/DarkYellow</material>
+            <minDepth>0.001</minDepth>
+            <!-- <implicitSpringDamper>1</implicitSpringDamper>
+            <springStiffness>100</springStiffness> -->
         </gazebo>
         <gazebo reference="${prefix}FL_FOOT">
-            <!-- <turnGravityOff>false</turnGravityOff>
-            <selfCollide>true</selfCollide>
-            <kp value="10000000.0"/>
-            <kd value="1.0"/>
-            <fdir1 value="1 0 0"/> -->
-            <mu1 value="0.2"/>
-            <mu2 value="0.2"/>
-            <material>Gazebo/Grey</material>
+            <mu1>0.9</mu1>
+            <mu2>0.9</mu2>
+            <fdir1>1 1 0</fdir1>
+            <kp value="2147483647.0" />
+            <kd value="100.0" />
+            <maxVel>0.01</maxVel>
+            <self_collide>1</self_collide>
+            <minDepth>0.001</minDepth>
+            <restitution_coefficient>1</restitution_coefficient>
+            <threshold>0</threshold>
+            <material>Gazebo/DarkGrey</material>
         </gazebo>
         <gazebo reference="${prefix}FR_SHOULDER">
-            <!-- <turnGravityOff>false</turnGravityOff>
-            <selfCollide>true</selfCollide>
-            <kp value="10000000.0"/>
-            <kd value="1.0"/>
-            <fdir1 value="1 0 0"/> -->
-            <mu1 value="0.2"/>
-            <mu2 value="0.2"/>
-            <material>Gazebo/Grey</material>
+            <mu1>0.2</mu1>
+            <mu2>0.2</mu2>
+            <kp value="2147483647.0"/>
+            <kd value="1.0"/>
+            <maxVel>0.01</maxVel>
+            <self_collide>1</self_collide>
+            <material>Gazebo/PioneerBody</material>
         </gazebo>
         <gazebo reference="${prefix}FR_UPPER_LEG">
-            <!-- <turnGravityOff>false</turnGravityOff>
-            <selfCollide>true</selfCollide>
-            <kp value="10000000.0"/>
-            <kd value="1.0"/>
-            <fdir1 value="1 0 0"/> -->
-            <mu1 value="0.2"/>
-            <mu2 value="0.2"/>
-            <material>Gazebo/Grey</material>
+            <mu1>0.2</mu1>
+            <mu2>0.2</mu2>
+            <kp value="2147483647.0"/>
+            <kd value="1.0"/>
+            <maxVel>0.01</maxVel>
+            <self_collide>1</self_collide>
+            <material>Gazebo/Orange</material>
+            <!-- <implicitSpringDamper>1</implicitSpringDamper>
+            <springStiffness>100</springStiffness> -->
         </gazebo>
         <gazebo reference="${prefix}FR_LOWER_LEG">
-            <!-- <turnGravityOff>false</turnGravityOff>
-            <selfCollide>true</selfCollide>
-            <kp value="10000000.0"/>
-            <kd value="1.0"/>
-            <fdir1 value="1 0 0"/> -->
-            <mu1 value="0.2"/>
-            <mu2 value="0.2"/>
-            <material>Gazebo/Grey</material>
+            <mu1>0.2</mu1>
+            <mu2>0.2</mu2>
+            <fdir1>1 0 0</fdir1>
+            <kp>2147483647.0</kp>
+            <kd>1.0</kd>
+            <maxVel>0.01</maxVel>
+            <self_collide>1</self_collide>
+            <material>Gazebo/DarkYellow</material>
+            <minDepth>0.001</minDepth>
+            <!-- <implicitSpringDamper>1</implicitSpringDamper>
+            <springStiffness>100</springStiffness> -->
         </gazebo>
         <gazebo reference="${prefix}FR_FOOT">
-            <!-- <turnGravityOff>false</turnGravityOff>
-            <selfCollide>true</selfCollide>
-            <kp value="10000000.0"/>
-            <kd value="1.0"/>
-            <fdir1 value="1 0 0"/> -->
-            <mu1 value="0.2"/>
-            <mu2 value="0.2"/>
-            <material>Gazebo/Grey</material>
+            <mu1>0.9</mu1>
+            <mu2>0.9</mu2>
+            <fdir1>1 1 0</fdir1>
+            <kp value="2147483647.0" />
+            <kd value="100.0" />
+            <maxVel>0.01</maxVel>
+            <self_collide>1</self_collide>
+            <minDepth>0.001</minDepth>
+            <restitution_coefficient>1</restitution_coefficient>
+            <threshold>0</threshold>
+            <material>Gazebo/DarkGrey</material>
         </gazebo>
         <gazebo reference="${prefix}HL_SHOULDER">
-            <!-- <turnGravityOff>false</turnGravityOff>
-            <selfCollide>true</selfCollide>
-            <kp value="10000000.0"/>
-            <kd value="1.0"/>
-            <fdir1 value="1 0 0"/> -->
-            <mu1 value="0.2"/>
-            <mu2 value="0.2"/>
-            <material>Gazebo/Grey</material>
+            <mu1>0.2</mu1>
+            <mu2>0.2</mu2>
+            <kp value="2147483647.0"/>
+            <kd value="1.0"/>
+            <maxVel>0.01</maxVel>
+            <self_collide>1</self_collide>
+            <material>Gazebo/PioneerBody</material>
         </gazebo>
         <gazebo reference="${prefix}HL_UPPER_LEG">
-            <!-- <turnGravityOff>false</turnGravityOff>
-            <selfCollide>true</selfCollide>
-            <kp value="10000000.0"/>
-            <kd value="1.0"/>
-            <fdir1 value="1 0 0"/> -->
-            <mu1 value="0.2"/>
-            <mu2 value="0.2"/>
-            <material>Gazebo/Grey</material>
+            <mu1>0.2</mu1>
+            <mu2>0.2</mu2>
+            <kp value="2147483647.0"/>
+            <kd value="1.0"/>
+            <maxVel>0.01</maxVel>
+            <self_collide>1</self_collide>
+            <material>Gazebo/Orange</material>
+            <!-- <implicitSpringDamper>1</implicitSpringDamper>
+            <springStiffness>100</springStiffness> -->
         </gazebo>
         <gazebo reference="${prefix}HL_LOWER_LEG">
-            <!-- <turnGravityOff>false</turnGravityOff>
-            <selfCollide>true</selfCollide>
-            <kp value="10000000.0"/>
-            <kd value="1.0"/>
-            <fdir1 value="1 0 0"/> -->
-            <mu1 value="0.2"/>
-            <mu2 value="0.2"/>
-            <material>Gazebo/Grey</material>
+            <mu1>0.2</mu1>
+            <mu2>0.2</mu2>
+            <fdir1>1 0 0</fdir1>
+            <kp>2147483647.0</kp>
+            <kd>1.0</kd>
+            <maxVel>0.01</maxVel>
+            <self_collide>1</self_collide>
+            <material>Gazebo/DarkYellow</material>
+            <minDepth>0.001</minDepth>
+            <!-- <implicitSpringDamper>1</implicitSpringDamper>
+            <springStiffness>100</springStiffness> -->
         </gazebo>
         <gazebo reference="${prefix}HL_FOOT">
-            <!-- <turnGravityOff>false</turnGravityOff>
-            <selfCollide>true</selfCollide>
-            <kp value="10000000.0"/>
-            <kd value="1.0"/>
-            <fdir1 value="1 0 0"/> -->
-            <mu1 value="0.2"/>
-            <mu2 value="0.2"/>
-            <material>Gazebo/Grey</material>
+            <mu1>0.9</mu1>
+            <mu2>0.9</mu2>
+            <fdir1>1 1 0</fdir1>
+            <kp value="2147483647.0" />
+            <kd value="100.0" />
+            <maxVel>0.01</maxVel>
+            <self_collide>1</self_collide>
+            <minDepth>0.001</minDepth>
+            <restitution_coefficient>1</restitution_coefficient>
+            <threshold>0</threshold>
+            <material>Gazebo/DarkGrey</material>
         </gazebo>
         <gazebo reference="${prefix}HR_SHOULDER">
-            <!-- <turnGravityOff>false</turnGravityOff>
-            <selfCollide>true</selfCollide>
-            <kp value="10000000.0"/>
-            <kd value="1.0"/>
-            <fdir1 value="1 0 0"/> -->
-            <mu1 value="0.2"/>
-            <mu2 value="0.2"/>
-            <material>Gazebo/Grey</material>
+            <mu1>0.2</mu1>
+            <mu2>0.2</mu2>
+            <kp value="2147483647.0"/>
+            <kd value="1.0"/>
+            <maxVel>0.01</maxVel>
+            <self_collide>1</self_collide>
+            <material>Gazebo/PioneerBody</material>
         </gazebo>
         <gazebo reference="${prefix}HR_UPPER_LEG">
-            <!-- <turnGravityOff>false</turnGravityOff>
-            <selfCollide>true</selfCollide>
-            <kp value="10000000.0"/>
-            <kd value="1.0"/>
-            <fdir1 value="1 0 0"/> -->
-            <mu1 value="0.2"/>
-            <mu2 value="0.2"/>
-            <material>Gazebo/Grey</material>
+            <mu1>0.2</mu1>
+            <mu2>0.2</mu2>
+            <kp value="2147483647.0"/>
+            <kd value="1.0"/>
+            <maxVel>0.01</maxVel>
+            <self_collide>1</self_collide>
+            <material>Gazebo/Orange</material>
+            <!-- <implicitSpringDamper>1</implicitSpringDamper>
+            <springStiffness>100</springStiffness> -->
         </gazebo>
         <gazebo reference="${prefix}HR_LOWER_LEG">
-            <!-- <turnGravityOff>false</turnGravityOff>
-            <selfCollide>true</selfCollide>
-            <kp value="10000000.0"/>
-            <kd value="1.0"/>
-            <fdir1 value="1 0 0"/> -->
-            <mu1 value="0.2"/>
-            <mu2 value="0.2"/>
-            <material>Gazebo/Grey</material>
+            <mu1>0.2</mu1>
+            <mu2>0.2</mu2>
+            <fdir1>1 0 0</fdir1>
+            <kp>2147483647.0</kp>
+            <kd>1.0</kd>
+            <maxVel>0.01</maxVel>
+            <self_collide>1</self_collide>
+            <material>Gazebo/DarkYellow</material>
+            <minDepth>0.001</minDepth>
+            <!-- <implicitSpringDamper>1</implicitSpringDamper>
+            <springStiffness>100</springStiffness> -->
         </gazebo>
         <gazebo reference="${prefix}HR_FOOT">
-            <!-- <turnGravityOff>false</turnGravityOff>
-            <selfCollide>true</selfCollide>
-            <kp value="10000000.0"/>
-            <kd value="1.0"/>
-            <fdir1 value="1 0 0"/> -->
-            <mu1 value="0.2"/>
-            <mu2 value="0.2"/>
-            <material>Gazebo/Grey</material>
+            <mu1>0.9</mu1>
+            <mu2>0.9</mu2>
+            <fdir1>1 1 0</fdir1>
+            <kp value="2147483647.0" />
+            <kd value="100.0" />
+            <maxVel>0.01</maxVel>
+            <self_collide>1</self_collide>
+            <minDepth>0.001</minDepth>
+            <restitution_coefficient>1</restitution_coefficient>
+            <threshold>0</threshold>
+            <material>Gazebo/DarkGrey</material>
         </gazebo>
     </xacro:macro>
