Commit message: corrected urdf; added dummy_link to base_link

File: solo12_description/urdf/solo12.urdf.xacro (robot description, xacro)
@@ -1,13 +1,11 @@
 <?xml version="1.0"?>
 <robot xmlns:xacro="http://www.ros.org/wiki/xacro">
-    <xacro:macro name="solo12_quadruped" params="prefix">
+    <xacro:macro name="solo12_quadruped" params="parent prefix">
         <!--The root link ${prefix}base_link has an inertia specified in
             the URDF, but KDL does not support a root link with an inertia.
             As a workaround, you can add an extra dummy link to your URDF.-->
-        <link name="world" />
-        <joint name="world_joint" type="fixed">
-            <parent link="world" />
+        <joint name="${prefix}dummy_joint" type="fixed">
+            <parent link="${parent}" />
             <child link="${prefix}base_link" />
-            <origin rpy="0 0 0" xyz="0 0 0" />
         </joint>
         <link name="${prefix}base_link">

Commit message: joint dynamics parameters modified

File: solo12_description/urdf/solo12.urdf.xacro (robot description, xacro)
@@ -55,5 +55,5 @@
             <origin rpy="0 0 0" xyz="0.1946 0.0875 0" />
             <!-- pybullet simulation parameters -->
-            <dynamics damping="0.0" friction="0.0" />
+            <dynamics damping="0.01" friction="10000"/>
         </joint>
         <link name="${prefix}FL_SHOULDER">
@@ -98,5 +98,5 @@
             <origin rpy="0 0 0" xyz="0 0.014 0" />
             <!-- pybullet simulation parameters -->
-            <dynamics damping="0.0" friction="0.0" />
+            <dynamics damping="0.01" friction="10000"/>
         </joint>
         <link name="${prefix}FL_UPPER_LEG">
@@ -146,5 +146,5 @@
             <origin rpy="0 0 0" xyz="0 0.03745 -0.16" />
             <!-- pybullet simulation parameters -->
-            <dynamics damping="0.0" friction="0.0" />
+            <dynamics damping="0.01" friction="10000"/>
         </joint>
         <link name="${prefix}FL_LOWER_LEG">
@@ -193,5 +193,5 @@
             <limit effort="1000" lower="-10" upper="10" velocity="1000" />
             <!-- pybullet simulation parameters -->
-            <dynamics damping="0.0" friction="0.0" />
+            <dynamics damping="0.01" friction="10000"/>
         </joint>
         <link name="${prefix}FL_FOOT">
@@ -241,5 +241,5 @@
             <origin rpy="0 0 0" xyz="0.1946 -0.0875 0" />
             <!-- pybullet simulation parameters -->
-            <dynamics damping="0.0" friction="0.0" />
+            <dynamics damping="0.01" friction="10000"/>
         </joint>
         <link name="${prefix}FR_SHOULDER">
@@ -284,5 +284,5 @@
             <origin rpy="0 0 0" xyz="0 -0.014 0" />
             <!-- pybullet simulation parameters -->
-            <dynamics damping="0.0" friction="0.0" />
+            <dynamics damping="0.01" friction="10000"/>
         </joint>
         <link name="${prefix}FR_UPPER_LEG">
@@ -332,5 +332,5 @@
             <origin rpy="0 0 0" xyz="0 -0.03745 -0.16" />
             <!-- pybullet simulation parameters -->
-            <dynamics damping="0.0" friction="0.0" />
+            <dynamics damping="0.01" friction="10000"/>
         </joint>
         <link name="${prefix}FR_LOWER_LEG">
@@ -379,5 +379,5 @@
             <limit effort="1000" lower="-10" upper="10" velocity="1000" />
             <!-- pybullet simulation parameters -->
-            <dynamics damping="0.0" friction="0.0" />
+            <dynamics damping="0.01" friction="10000"/>
         </joint>
         <link name="${prefix}FR_FOOT">
@@ -427,5 +427,5 @@
             <origin rpy="0 0 0" xyz="-0.1946 0.0875 0" />
             <!-- pybullet simulation parameters -->
-            <dynamics damping="0.0" friction="0.0" />
+            <dynamics damping="0.01" friction="10000"/>
         </joint>
         <link name="${prefix}HL_SHOULDER">
@@ -470,5 +470,5 @@
             <origin rpy="0 0 0" xyz="0 0.014 0" />
             <!-- pybullet simulation parameters -->
-            <dynamics damping="0.0" friction="0.0" />
+            <dynamics damping="0.01" friction="10000"/>
         </joint>
         <link name="${prefix}HL_UPPER_LEG">
@@ -518,5 +518,5 @@
             <origin rpy="0 0 0" xyz="0 0.03745 -0.16" />
             <!-- pybullet simulation parameters -->
-            <dynamics damping="0.0" friction="0.0" />
+            <dynamics damping="0.01" friction="10000"/>
         </joint>
         <link name="${prefix}HL_LOWER_LEG">
@@ -565,5 +565,5 @@
             <limit effort="1000" lower="-10" upper="10" velocity="1000" />
             <!-- pybullet simulation parameters -->
-            <dynamics damping="0.0" friction="0.0" />
+            <dynamics damping="0.01" friction="10000"/>
         </joint>
         <link name="${prefix}HL_FOOT">
@@ -613,5 +613,5 @@
             <origin rpy="0 0 0" xyz="-0.1946 -0.0875 0" />
             <!-- pybullet simulation parameters -->
-            <dynamics damping="0.0" friction="0.0" />
+            <dynamics damping="0.01" friction="10000"/>
         </joint>
         <link name="${prefix}HR_SHOULDER">
@@ -656,5 +656,5 @@
             <origin rpy="0 0 0" xyz="0 -0.014 0" />
             <!-- pybullet simulation parameters -->
-            <dynamics damping="0.0" friction="0.0" />
+            <dynamics damping="0.01" friction="10000"/>
         </joint>
         <link name="${prefix}HR_UPPER_LEG">
@@ -704,5 +704,5 @@
             <origin rpy="0 0 0" xyz="0 -0.03745 -0.16" />
             <!-- pybullet simulation parameters -->
-            <dynamics damping="0.0" friction="0.0" />
+            <dynamics damping="0.01" friction="10000"/>
         </joint>
         <link name="${prefix}HR_LOWER_LEG">
@@ -751,5 +751,5 @@
             <limit effort="1000" lower="-10" upper="10" velocity="1000" />
             <!-- pybullet simulation parameters -->
-            <dynamics damping="0.0" friction="0.0" />
+            <dynamics damping="0.01" friction="10000"/>
         </joint>
         <link name="${prefix}HR_FOOT">
